Commit message: 新版模型顶层设计和直线运行模式修复

File: ice_cream_SINGLE.SLDASM/urdf/ice_cream_SINGLE.SLDASM.urdf (robot description, URDF)
Before this commit: robot ice_cream_SINGLE.SLDASM, 8 links, 7 joints
Joints:
- joint FINGER_RIGHT: axis 0 0 0 -> 0 0 -1
- joint joint1: axis 0 0 0 -> 0 0 -1
- joint joint2: axis 0 0 0 -> 0 0 -1
- joint joint3: axis 0 0 0 -> 0 0 -1
- joint joint4: axis 0 0 0 -> 0 0 -1
- joint joint5: axis 0 0 0 -> 0 0 -1
